Commit message: Add controller to joint

File: robots/lumyai.xacro (robot description, xacro)
@@ -1,5 +1,4 @@
 <?xml version="1.0"?>
 <robot name="lumyai_neli" xmlns:xacro="http://www.ros.org/wiki/xacro">
-    <xacro:include filename="$(find lumyai_descriptions)/robots/lumyai_neli.URDF" />
     <gazebo>
         <plugin name="object_controller" filename="libgazebo_ros_planar_move.so">
@@ -24,7 +23,4 @@
             </geometry>
         </collision>
-        <visual>
-            <origin xyz="0 0 0" rpy="0 0 0"/>
-        </visual>
         <inertial>
             <mass value="1e-5" />
@@ -60,5 +56,5 @@
                             reading. -->
                     <mean>0.0</mean>
-                    <stddev>0.01</stddev>
+                    <stddev>0.005</stddev>
                 </noise>
             </ray>
@@ -69,3 +65,37 @@
         </sensor>
     </gazebo>
+    <gazebo>
+        <plugin name="gazebo_ros_control" filename="libgazebo_ros_control.so">
+            <robotNamespace>/lumyai_neli</robotNamespace>
+        </plugin>
+    </gazebo>
+    <xacro:macro name="joint_motor" params="joint_name id">
+        <transmission name="tran_${joint_name}">
+            <type>transmission_interface/SimpleTransmission</type>
+            <joint name="${joint_name}">
+                <hardwareInterface>EffortJointInterface</hardwareInterface>
+            </joint>
+            <actuator name="motor_${id}">
+                <hardwareInterface>EffortJointInterface</hardwareInterface>
+                <mechanicalReduction>1</mechanicalReduction>
+            </actuator>
+        </transmission>
+    </xacro:macro>
+    <xacro:joint_motor joint_name="pan_joint" id="10"/>
+    <xacro:joint_motor joint_name="tilt_joint" id="11"/>
+    <xacro:joint_motor joint_name="right_shoulder_1_joint" id="30"/>
+    <xacro:joint_motor joint_name="right_shoulder_2_joint" id="31"/>
+    <xacro:joint_motor joint_name="right_elbow_joint" id="32"/>
+    <xacro:joint_motor joint_name="right_wrist_1_joint" id="40"/>
+    <xacro:joint_motor joint_name="right_wrist_2_joint" id="41"/>
+    <xacro:joint_motor joint_name="right_wrist_3_joint" id="42"/>
+    <xacro:joint_motor joint_name="right_gripper_joint" id="43"/>
+    <xacro:joint_motor joint_name="left_shoulder_1_joint" id="35"/>
+    <xacro:joint_motor joint_name="left_shoulder_2_joint" id="36"/>
+    <xacro:joint_motor joint_name="left_elbow_joint" id="37"/>
+    <xacro:joint_motor joint_name="left_wrist_1_joint" id="45"/>
+    <xacro:joint_motor joint_name="left_wrist_2_joint" id="46"/>
+    <xacro:joint_motor joint_name="left_wrist_3_joint" id="47"/>
+    <xacro:joint_motor joint_name="left_gripper_joint" id="48"/>
+    <xacro:include filename="$(find lumyai_descriptions)/robots/lumyai_neli.URDF" />
 </robot>

Commit message: Tuning PID for all manipulators

File: robots/lumyai.xacro (robot description, xacro)
@@ -9,59 +9,4 @@
             <robotBaseFrame>base_link</robotBaseFrame>
         </plugin>
-    </gazebo>
-    <joint name="hokuyo_joint" type="fixed">
-        <axis xyz="0 1 0"/>
-        <origin xyz="0 0 0.05" rpy="0 0 0"/>
-        <parent link="laser_Link"/>
-        <child link="hokuyo_link"/>
-    </joint>
-    <link name="hokuyo_link">
-        <collision>
-            <origin xyz="0 0 0" rpy="0 0 0"/>
-            <geometry>
-                <box size="0.1 0.1 0.1"/>
-            </geometry>
-        </collision>
-        <inertial>
-            <mass value="1e-5" />
-            <origin xyz="0 0 0" rpy="0 0 0"/>
-            <inertia ixx="1e-6" ixy="0" ixz="0" iyy="1e-6" iyz="0" izz="1e-6" />
-        </inertial>
-    </link>
-    <!-- hokuyo -->
-    <gazebo reference="hokuyo_link">
-        <sensor type="ray" name="hokuyo_sensor">
-            <pose>0 0 0 0 0 0</pose>
-            <visualize>false</visualize>
-            <update_rate>30</update_rate>
-            <ray>
-                <scan>
-                    <horizontal>
-                        <samples>720</samples>
-                        <resolution>1</resolution>
-                        <min_angle>-1.570796</min_angle>
-                        <max_angle>1.570796</max_angle>
-                    </horizontal>
-                </scan>
-                <range>
-                    <min>0.10</min>
-                    <max>30.0</max>
-                    <resolution>0.01</resolution>
-                </range>
-                <noise>
-                    <type>gaussian</type>
-                        <!-- Noise parameters based on published spec for Hokuyo laser
-                            achieving "+-30mm" accuracy at range < 10m.  A mean of 0.0m and
-                            stddev of 0.01m will put 99.7% of samples within 0.03m of the true
-                            reading. -->
-                    <mean>0.0</mean>
-                    <stddev>0.005</stddev>
-                </noise>
-            </ray>
-            <plugin name="gazebo_ros_hokuyo_controller" filename="libgazebo_ros_laser.so">
-                <topicName>/laser/scan</topicName>
-                <frameName>laser_Link</frameName>
-            </plugin>
-        </sensor>
     </gazebo>
     <gazebo>
@@ -99,3 +44,4 @@
     <xacro:joint_motor joint_name="left_gripper_joint" id="48"/>
     <xacro:include filename="$(find lumyai_descriptions)/robots/lumyai_neli.URDF" />
+    <xacro:include filename="$(find athome_simulation)/robots/sensors.xacro" />
 </robot>
